File: TP1213.kicad_sch (KiCad schematic)
At the start: 0 parts

Commit message: add sheet setting
Other:
- company: (none) -> @stop-pattern
- title: (none) -> TP1213
Changed lines of the file:
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@@
 	(generator_version "8.0")
 	(paper "A4")
+	(title_block
+		(title "TP1213")
+		(date "2025-01-14")
+		(rev "0.00")
+		(company "@stop-pattern")
+		(comment 4 "汎用ジョイスティック基板")
+	)
 	(sheet_instances
 		(path "/"
